File: board_design/Connect-Stethoscope.kicad_sch (KiCad schematic)
At the start: 3 parts, among them M0 Motor_Servo

Commit message: Wiring diagrams
Parts:
- removed J?: Conn_01x05_Female, symbol Connector:Conn_01x05_Female
- removed M0: Motor_Servo, symbol Motor:Motor_Servo
- added J1: Conn_01x05, Connector_PinSocket_2.54mm:PinSocket_1x05_P2.54mm_Horizontal, symbol Connector_Generic:Conn_01x05
- added J2: Conn_01x03, Connector:Banana_Jack_3Pin, symbol Connector_Generic:Conn_01x03
- added M1, M2: Motor_Servo, Connector_PinHeader_2.54mm:PinHeader_1x03_P2.54mm_Vertical, symbol Motor:Motor_Servo
- U1: renamed from U?; footprint RPi_Pico:RPi_Pico_SMD_TH -> MCU_RaspberryPi_and_Boards:RPi_Pico_SMD_TH
Connections:
- net at U1.27 (GPIO21): now also J1.5 (Pin_5)
- net VBUS: now reaches U1.40 (VBUS)
- net VBUS: now also M1.2 (+), M2.2 (+)
- net GND: now reaches U1.38 (GND)
- net GND: now also U1.13 (GND), U1.18 (GND), U1.23 (GND), U1.28 (GND), U1.3 (GND), U1.8 (GND), J1.1 (Pin_1), J2.2 (Pin_2), M1.3 (-), M2.3 (-)
- net at U1.11 (GPIO8): now also J2.3 (Pin_3)
- net at U1.12 (GPIO9): now also J2.1 (Pin_1)
- net at U1.29 (GPIO22): now also J1.4 (Pin_4)
- net at U1.31 (GPIO26_ADC0): now also J1.3 (Pin_3)
- net +3V3: now reaches U1.36 (3V3)
- net +3V3: now also J1.2 (Pin_2)
- net at U1.4 (GPIO2): now also M1.1 (PWM)
- net at U1.5 (GPIO3): now also M2.1 (PWM)
